File: TeensyluV1/Teensylu-1.1.brd (EAGLE design)
At the start: 101.6 x 76.2 mm, 101 parts, among them J1 M02POLAR, J11 M02POLAR, J12 M02POLAR, J2 MICROSD, J3 USB-MICRO-PTH, J4 M02POLAR, J5 4P-TERM-BLOCK284391-4, J6 39-29-3066, J7 HOTEND-1, J8 2x7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

Commit message: Fixed Z endstop
Collector and emitter pins were swapped.
Connections:
- net GND: now also Q5.2; no longer Q5.3
- net Z-STOP: now also Q5.3; no longer Q5.2
Other:
- board text added: "Rev. 1.1"
- board text added: "https://github.com/StephS/Teensylu"
- board text removed: "Rev. 1.0"
- board text removed: "https://github.com/StephS/Teensylu2"
Changed lines of the file:
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@@
 <text x="48.26" y="10.922" size="0.8128" layer="121" font="vector" ratio="15" rot="R180">+12V</text>
 <text x="62.738" y="30.734" size="1.27" layer="121" font="vector" ratio="15">TeensyluV1</text>
-<text x="62.738" y="28.956" size="1.27" layer="121" font="vector" ratio="15">Rev. 1.0</text>
-<text x="62.738" y="27.432" size="1.016" layer="121" font="vector" ratio="15">https://github.com/StephS/Teensylu2</text>
+<text x="62.738" y="28.956" size="1.27" layer="121" font="vector" ratio="15">Rev. 1.1</text>
+<text x="62.738" y="27.432" size="1.016" layer="121" font="vector" ratio="15">https://github.com/StephS/Teensylu</text>
 <text x="62.738" y="25.908" size="1.016" layer="121" font="vector" ratio="15">Licensed CC-BY-SA</text>
 <text x="38.354" y="6.096" size="1.016" layer="121" font="vector" ratio="15">Z-STOP</text>
@@
 <via x="31.242" y="29.718" extent="1-16" drill="0.4"/>
 <via x="95.25" y="53.086" extent="1-16" drill="0.4"/>
-<contactref element="Q5" pad="3"/>
 <via x="28.956" y="60.452" extent="1-16" drill="0.4"/>
 <via x="49.276" y="60.452" extent="1-16" drill="0.4"/>
@@
 <via x="22.352" y="20.828" extent="1-16" drill="0.4"/>
 <via x="22.352" y="19.304" extent="1-16" drill="0.4"/>
+<contactref element="Q5" pad="2"/>
 </signal>
 <signal name="!RESET">
@@
 </signal>
 <signal name="Z-STOP">
-<wire x1="43.18" y1="18.4843125" x2="43.18" y2="16.256" width="0.254" layer="1"/>
-<contactref element="Q5" pad="2"/>
-<wire x1="43.18" y1="16.256" x2="43.368" y2="15.682" width="0.254" layer="1"/>
-<wire x1="43.368" y1="15.682" x2="43.264" y2="15.682" width="0.254" layer="1"/>
+<wire x1="41.148" y1="18.4843125" x2="41.148" y2="17.018" width="0.254" layer="1"/>
 <contactref element="U5" pad="1"/>
+<wire x1="41.148" y1="17.018" x2="41.148" y2="16.764" width="0.254" layer="1"/>
 <wire x1="41.041925" y1="27.93720625" x2="39.878" y2="26.77328125" width="0.254" layer="1"/>
 <wire x1="39.878" y1="26.77328125" x2="39.878" y2="26.67" width="0.254" layer="1"/>
 <via x="39.878" y="26.67" extent="1-16" drill="0.4"/>
-<wire x1="39.878" y1="26.67" x2="39.878" y2="21.7863125" width="0.254" layer="16"/>
-<wire x1="39.878" y1="21.7863125" x2="43.18" y2="18.4843125" width="0.254" layer="16"/>
-<via x="43.18" y="18.4843125" extent="1-16" drill="0.4"/>
+<wire x1="39.878" y1="26.67" x2="39.878" y2="19.7543125" width="0.254" layer="16"/>
+<wire x1="39.878" y1="19.7543125" x2="41.148" y2="18.4843125" width="0.254" layer="16"/>
+<via x="41.148" y="18.4843125" extent="1-16" drill="0.4"/>
+<contactref element="Q5" pad="3"/>
+<wire x1="41.064" y1="14.732" x2="41.148" y2="14.732" width="0.254" layer="1"/>
+<wire x1="41.148" y1="14.732" x2="41.148" y2="16.764" width="0.254" layer="1"/>
 </signal>
 <signal name="X-STEP">
@@
 <contactref element="JP7" pad="1"/>
 <contactref element="Q5" pad="1"/>
-<wire x1="43.264" y1="13.782" x2="45.212" y2="11.834" width="0.254" layer="1"/>
 <wire x1="45.212" y1="11.834" x2="45.212" y2="4.826" width="0.254" layer="1"/>
 <wire x1="45.212" y1="4.826" x2="43.688" y2="3.302" width="0.254" layer="1"/>
+<wire x1="43.264" y1="13.782" x2="45.212" y2="11.834" width="0.254" layer="1"/>
 </signal>
 <signal name="PE3">
