File: TeensyluV1-2Layer/Teensylu-1.3a.sch (EAGLE design)
At the start: 110 parts, among them J1 22ga, J10 MICROSD, J11 USB-MICRO-PTH, J12 M02POLAR, J13 4P-TERM-BLOCK284391-4, J14 HOTEND-1, J15 39-29-3066, J16 2x7, J17 HOTBED, J18 M02POLAR, J19 M02POLAR, J2 22ga, J3 22ga, J4 22ga, J5 22ga, J6 22ga, J7 22ga, J8 M02POLAR, J9 M02POLAR, P1 POLOLU-X, P2 POLOLU-Y, P3 POLOLU-Z, P4 POLOLU-E1, Q1 PMV45EN, Q2 PSMN1R2-30YLC, Q3 MMUN2211LT3G, Q4 PSMN1R2-30YLC, U1 LMR16006X, U2 DRTR5V0U2SR, U3 AP7313SOT23C, U4 TXB0104TSSOP14, U5 AT90USB1286, X1 16MHZ

Commit message: Updated heater mosfets
I updated the heater mosfets to 40v version, part # PSMN1R8-40YLC,115
Parts:
- Q2, Q4: value PSMN1R2-30YLC -> PSMN1R8-40YLC; device teensylu:PSMN1R2-30YLCPOWERPACK-S08 -> teensylu:PSMN1R8-40YLCPOWERPACK-S08
Other:
- note added: "Rev 1.3a"
- note removed: "Rev 1.3"
Changed lines of the file:
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@@
 <attribute name="VDC" value="16V"/>
 </part>
-<part name="Q2" library="teensylu" deviceset="PSMN1R2-30YLC" device="POWERPACK-S08" value="PSMN1R2-30YLC"/>
-<part name="Q4" library="teensylu" deviceset="PSMN1R2-30YLC" device="POWERPACK-S08" value="PSMN1R2-30YLC"/>
+<part name="Q2" library="teensylu" deviceset="PSMN1R8-40YLC" device="POWERPACK-S08" value="PSMN1R8-40YLC"/>
+<part name="Q4" library="teensylu" deviceset="PSMN1R8-40YLC" device="POWERPACK-S08" value="PSMN1R8-40YLC"/>
 <part name="SJ10" library="teensylu" deviceset="SOLDERJUMPER-NC" device="SJ-TRACE" value="MS1"/>
 <part name="SJ6" library="teensylu" deviceset="SOLDERJUMPER-NC" device="SJ-TRACE" value="MS2"/>
@@
 <text x="2.54" y="154.94" size="1.778" layer="91" font="vector">Power Acc</text>
 <text x="60.96" y="7.62" size="3.81" layer="94">TeensyluV1</text>
-<text x="175.26" y="7.62" size="2.54" layer="94">Rev 1.3</text>
+<text x="175.26" y="7.62" size="2.54" layer="94">Rev 1.3a</text>
 <text x="111.76" y="7.62" size="3.048" layer="94">Control for Reprap</text>
 <text x="63.5" y="2.54" size="2.032" layer="94">Licensed under the Creative Commons Attributions ShareAlike 3.0 License</text>
